File: hackpad.kicad_sch (KiCad schematic)
At the start: 7 parts, among them SW0 SW_Push, SW1 SW_Push, SW2 SW_Push, SW3 SW_Push, U1 XIAO-RP2040-DIP

Commit message: Do more stuff & Add gitignore & pcb stuff.
Parts:
- SW0, SW1, SW2, SW3: footprint (none) -> Button_Switch_Keyboard:SW_Cherry_MX_1.00u_PCB
- U1: footprint Module:MOUDLE14P-XIAO-DIP-SMD -> Seeed Studio XIAO Series Library:XIAO-RP2040-DIP
Connections:
- net GND: now reaches D2.2 (VSS)
- net GND: now also D1.2 (VSS), U1.13 (GND)
- net at D2.3 (DIN): now also D1.1 (DOUT)
- net +5V: now reaches D2.4 (VDD)
- net +5V: now also D1.4 (VDD), U1.14 (VBUS)
- net at U1.10 (GPIO4/MISO): now also SW2.2
- net at U1.11 (GPIO3/MOSI): now also SW3.2
- net at U1.5 (GPIO6/SDA): now also D1.3 (DIN)
- net at U1.8 (GPIO1/RX): now also SW0.2
- net at U1.9 (GPIO2/SCK): now also SW1.2
