File: hackpad.kicad_pcb (KiCad board)
At the start: 2 copper layers, 7 parts, among them SW0 SW_Push, SW1 SW_Push, SW2 SW_Push, SW3 SW_Push, U1 XIAO-RP2040-DIP

Commit message: 幹，I don't like kicad, 我用到沒有耐心了，我也有強迫症，沒有對齊就更本做不下去啊
Parts:
- moved D2 56.3 mm to (201.8, 99.1)
- moved D1 56.1 mm to (171.4, 100.0)
- moved SW2 40.5 mm to (178.6, 130.7)
- moved SW3 38.3 mm to (200.5, 130.7)
- moved SW1 15.1 mm to (199.9, 109.2)
- moved SW0 12.6 mm to (178.6, 109.2)
- moved U1 12.4 mm to (185.3, 92.4)
Connections:
- SW0 pad 1: Net-(SW0-Pad1) -> GND
- SW1 pad 1: Net-(SW0-Pad1) -> GND
- SW2 pad 1: Net-(SW0-Pad1) -> GND
- SW3 pad 1: Net-(SW0-Pad1) -> GND
Routing:
- net GND: track 0.00 -> 103.9 mm
- net Net-(D1-DOUT): track 0.00 -> 60.2 mm
- net +5V: track 0.00 -> 45.9 mm
- net Net-(D1-DIN): track 0.00 -> 8.43 mm
Other:
- board outline added: 45.2 x 66.7 mm
